Commit message: Organize package structure and implement semantic object tracking

File: models/mecanum_bot.urdf (robot description, URDF)
Before this commit: robot robot, 9 links, 8 joints
Links:
- removed link camera_link
- removed link dustbin_body
- link back_left_wheel: mass 0.5 -> 0.15
- link back_right_wheel: mass 0.5 -> 0.15
- link base_link: mass 10.0 -> 1.2
- link front_left_wheel: mass 0.5 -> 0.15
- link front_right_wheel: mass 0.5 -> 0.15
- link laser_frame: mass 0.1 -> None; geometry collision cylinder length=0.01 radius=0.02; visual cylinder length=0.01 radius=0.02
Joints:
- removed joint camera_joint
- removed joint dustbin_joint
- joint back_left_wheel_joint: origin xyz=-0.15 0.12 0.0 rpy=1.5707 0 0 -> xyz=-0.1 0.12 -0.0275 rpy=1.5707 0 0
- joint back_right_wheel_joint: origin xyz=-0.15 -0.12 0.0 rpy=1.5707 0 0 -> xyz=-0.1 -0.12 -0.0275 rpy=1.5707 0 0
- joint base_joint: origin xyz=0 0 0.0325 rpy=0 0 0 -> xyz=0 0 0.06 rpy=0 0 0
- joint front_left_wheel_joint: origin xyz=0.15 0.12 0.0 rpy=1.5707 0 0 -> xyz=0.1 0.12 -0.0275 rpy=1.5707 0 0
- joint front_right_wheel_joint: origin xyz=0.15 -0.12 0.0 rpy=1.5707 0 0 -> xyz=0.1 -0.12 -0.0275 rpy=1.5707 0 0
- joint laser_joint: origin xyz=0 0 0.27 rpy=0 0 0 -> xyz=0.1 0 0.30 rpy=0 0 0
