Commit message: Enhance: Document project progress & integrate vision camera to URDF

File: models/robot_dual_arm.urdf (robot description, URDF)
Before this commit: robot robot, 17 links, 16 joints
Links:
- added link camera_link, mass 0.001; visual box size=0.02 0.04 0.02
Joints:
- added joint camera_joint: type fixed, parent base_link, child camera_link, origin xyz=0.13 0 0.08 rpy=0 0 0
